File: PCB/Bakers-dozen.sch (KiCad schematic (older format))
At the start: 114 parts, among them SW1 SW_Push, U1 ATmega32U4-AU, Y1 16Mhz

Commit message: Plate size and change footprint
Parts:
- MX1, MX10, MX11, MX12, MX13, MX14, MX15, MX16, MX17, MX18, MX19, MX2, MX20, MX21, MX22, MX23, MX24, MX25, MX26, MX27, MX28, MX29, MX3, MX30, MX31, MX32, MX33, MX34, MX35, MX36, MX37, MX38, MX39, MX4, MX40, MX41, MX42, MX43, MX45, MX47, MX48, MX49, MX5, MX6, MX7, MX8, MX9: footprint MX_Alps_Hybrid:MX-1U-NoLED -> MX_Alps_Hybrid:MX-1U
- MX44: footprint MX_Alps_Hybrid:MX-2.75U-NoLED -> MX_Alps_Hybrid:MX-2.75U
- MX46: footprint MX_Alps_Hybrid:MX-2.25U-NoLED -> MX_Alps_Hybrid:MX-2.25U

Commit message: Trace pcb
Parts:
- MX1, MX10, MX11, MX12, MX13, MX14, MX15, MX16, MX17, MX18, MX19, MX2, MX20, MX21, MX22, MX23, MX24, MX25, MX26, MX27, MX28, MX29, MX3, MX30, MX31, MX32, MX33, MX34, MX35, MX36, MX37, MX38, MX39, MX4, MX40, MX41, MX42, MX43, MX45, MX47, MX48, MX49, MX5, MX6, MX7, MX8, MX9: footprint MX_Alps_Hybrid:MX-1U -> MX_Alps_Hybrid:MX-1U-NoLED
- MX44: footprint MX_Alps_Hybrid:MX-2.75U -> MX_Alps_Hybrid:MX-2.75U-NoLED
- MX46: footprint MX_Alps_Hybrid:MX-2.25U -> MX_Alps_Hybrid:MX-2.25U-NoLED
