File: PCB/Bakers-dozen.sch (KiCad schematic (older format))
At the start: 114 parts, among them SW1 SW_Push, U1 ATmega32U4-AU, Y1 16Mhz

Commit message: Flip stabs
Parts:
- MX44: footprint MX_Alps_Hybrid:MX-2.75U-NoLED -> MX_Alps_Hybrid:MX-2.75U-ReversedStabilizers-NoLED
- MX46: footprint MX_Alps_Hybrid:MX-2.25U-NoLED -> MX_Alps_Hybrid:MX-2.25U-ReversedStabilizers-NoLED
Changed lines of the file:
@@
 F 0 "MX46" H 10283 6273 60  0000 C CNN
 F 1 "MX-NoLED" H 10283 6199 20  0000 C CNN
-F 2 "MX_Alps_Hybrid:MX-2.25U-NoLED" H 9625 6025 60  0001 C CNN
+F 2 "MX_Alps_Hybrid:MX-2.25U-ReversedStabilizers-NoLED" H 9625 6025 60  0001 C CNN
 F 3 "" H 9625 6025 60  0001 C CNN
 	1    10250 6050
@@
 F 0 "MX44" H 8783 6273 60  0000 C CNN
 F 1 "MX-NoLED" H 8783 6199 20  0000 C CNN
-F 2 "MX_Alps_Hybrid:MX-2.75U-NoLED" H 8125 6025 60  0001 C CNN
+F 2 "MX_Alps_Hybrid:MX-2.75U-ReversedStabilizers-NoLED" H 8125 6025 60  0001 C CNN
 F 3 "" H 8125 6025 60  0001 C CNN
 	1    8750 6050
