File: PCB/Bakers-dozen.kicad_pcb (KiCad board)
At the start: 2 copper layers, 247.7 x 81.8 mm, 114 parts, among them SW1 SW_Push, U1 ATmega32U4-AU, Y1 16Mhz

Commit message: Trace pcb
Parts:
- MX1, MX10, MX11, MX12, MX13, MX14, MX15, MX16, MX17, MX18, MX19, MX2, MX20, MX21, MX22, MX23, MX24, MX25, MX26, MX27, MX28, MX29, MX3, MX30, MX31, MX32, MX33, MX34, MX35, MX36, MX37, MX38, MX39, MX4, MX40, MX41, MX42, MX43, MX45, MX47, MX48, MX49, MX5, MX6, MX7, MX8, MX9: footprint MX_Alps_Hybrid:MX-1U -> MX_Alps_Hybrid:MX-1U-NoLED
- MX44: footprint MX_Alps_Hybrid:MX-2.75U -> MX_Alps_Hybrid:MX-2.75U-NoLED
- MX46: footprint MX_Alps_Hybrid:MX-2.25U -> MX_Alps_Hybrid:MX-2.25U-NoLED
- moved R1 98.2 mm to (136.5, 117.5)
- moved C6 3.27 mm to (160.3, 134.1), turned to 270 degrees
- moved C3 1.77 mm to (142.9, 129.4)
- moved D49 0.79 mm to (275.4, 127.0)
Routing:
- net ROW0: track 0.00 -> 434.8 mm, vias 0 -> 6
- net ROW1: track 0.00 -> 413.5 mm, vias 0 -> 4
- net ROW2: track 0.00 -> 392.9 mm, vias 0 -> 2
- net GND: track 0.00 -> 298.7 mm, vias 0 -> 6
- net +5V: track 0.00 -> 297.9 mm, vias 0 -> 7
- net COL0: track 0.00 -> 284.5 mm, vias 0 -> 4
- net COL1: track 0.00 -> 273.1 mm, vias 0 -> 4
- net COL2: track 0.00 -> 246.0 mm, vias 0 -> 3
- net ROW3: track 0.00 -> 237.3 mm, vias 0 -> 4
- net COL12: track 0.00 -> 237.1 mm, vias 0 -> 5
- net COL3: track 0.00 -> 219.2 mm, vias 0 -> 3
- net COL11: track 0.00 -> 215.9 mm, vias 0 -> 5
- net Net-(R4-Pad2): track 0.00 -> 199.2 mm, vias 0 -> 2
- net COL10: track 0.00 -> 193.8 mm, vias 0 -> 5
- net Net-(R3-Pad1): track 0.00 -> 153.4 mm, vias 0 -> 2
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Other:
- board size 247.7 x 81.8 mm -> 247.7 x 82.5 mm
- net class Power added: clearance 0.2, trace_width 0.38, via_dia 0.8, via_drill 0.4
- rule pad_to_mask_clearance: 0.051 -> 0.052

Commit message: Ground fills
Routing:
- net ROW3: track 237.3 -> 268.1 mm
- net +5V: track 297.9 -> 303.4 mm
- net COL0: track 284.5 -> 285.6 mm
- added copper zone on B.Cu, net (none)
- added copper zone on F.Cu, net (none)
Changed lines of the file:
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@@
     (thickness 1.6)
     (drawings 16)
-    (tracks 1049)
+    (tracks 1059)
     (zones 0)
     (modules 114)
@@
   (page A4)
   (layers
-    (0 F.Cu signal)
-    (31 B.Cu signal)
+    (0 F.Cu signal hide)
+    (31 B.Cu signal hide)
     (32 B.Adhes user)
     (33 F.Adhes user)
@@
   (segment (start 147.4875 126.20625) (end 147.49375 126.2) (width 0.38) (layer B.Cu) (net 5))
   (segment (start 144.4625 126.20625) (end 147.4875 126.20625) (width 0.38) (layer B.Cu) (net 5))
-  (segment (start 146.05 133.35) (end 144.4625 131.7625) (width 0.38) (layer F.Cu) (net 5))
   (segment (start 148.43125 135.73125) (end 146.05 133.35) (width 0.38) (layer F.Cu) (net 5))
   (via (at 146.05 130.96875) (size 0.8) (drill 0.4) (layers F.Cu B.Cu) (net 5))
@@
   (segment (start 162.71875 135.73125) (end 168.275 135.73125) (width 0.38) (layer F.Cu) (net 5))
   (segment (start 148.43125 135.73125) (end 162.71875 135.73125) (width 0.38) (layer F.Cu) (net 5))
+  (segment (start 146.05 133.35) (end 144.4625 131.7625) (width 0.38) (layer F.Cu) (net 5))
+  (segment (start 146.05 131.534435) (end 146.05 130.96875) (width 0.38) (layer B.Cu) (net 5))
+  (segment (start 146.05 132.56875) (end 146.05 131.534435) (width 0.38) (layer B.Cu) (net 5))
+  (segment (start 148.41875 134.9375) (end 146.05 132.56875) (width 0.38) (layer B.Cu) (net 5))
+  (segment (start 148.99375 134.9375) (end 148.41875 134.9375) (width 0.38) (layer B.Cu) (net 5))
   (segment (start 44.24375 68.2) (end 46.83125 68.2) (width 0.25) (layer B.Cu) (net 6))
   (segment (start 41.39375 65.35) (end 44.24375 68.2) (width 0.25) (layer B.Cu) (net 6))
@@
   (segment (start 273.912349 129.318901) (end 257.900151 129.318901) (width 0.25) (layer B.Cu) (net 49))
   (segment (start 275.43125 128.65) (end 274.58125 128.65) (width 0.25) (layer B.Cu) (net 49))
+  (segment (start 235.812349 129.318901) (end 236.48125 128.65) (width 0.25) (layer B.Cu) (net 49))
+  (segment (start 208.687651 129.318901) (end 235.812349 129.318901) (width 0.25) (layer B.Cu) (net 49))
+  (segment (start 236.48125 128.65) (end 237.33125 128.65) (width 0.25) (layer B.Cu) (net 49))
+  (segment (start 208.01875 128.65) (end 208.687651 129.318901) (width 0.25) (layer B.Cu) (net 49))
+  (segment (start 207.16875 128.65) (end 208.01875 128.65) (width 0.25) (layer B.Cu) (net 49))
   (segment (start 63.29375 125.35) (end 65.88125 125.35) (width 0.25) (layer B.Cu) (net 50))
   (segment (start 60.44375 122.5) (end 63.29375 125.35) (width 0.25) (layer B.Cu) (net 50))
@@
   (segment (start 186.53125 132.55625) (end 186.53125 130.96875) (width 0.25) (layer B.Cu) (net 60))
   (segment (start 186.53125 130.96875) (end 188.348501 129.151499) (width 0.25) (layer F.Cu) (net 60))
-  (segment (start 188.348501 129.151499) (end 188.348501 108.323049) (width 0.25) (layer F.Cu) (net 60))
-  (segment (start 184.872101 104.846649) (end 184.872101 96.115399) (width 0.25) (layer F.Cu) (net 60))
-  (segment (start 184.872101 104.846649) (end 184.800452 104.775) (width 0.25) (layer F.Cu) (net 60))
-  (segment (start 188.348501 108.323049) (end 184.872101 104.846649) (width 0.25) (layer F.Cu) (net 60))
   (via (at 184.94375 96.04375) (size 0.8) (drill 0.4) (layers F.Cu B.Cu) (net 60))
-  (segment (start 184.872101 96.115399) (end 184.94375 96.04375) (width 0.25) (layer F.Cu) (net 60))
   (segment (start 181.837499 92.937499) (end 38.031251 92.937499) (width 0.25) (layer B.Cu) (net 60))
   (segment (start 184.94375 96.04375) (end 181.837499 92.937499) (width 0.25) (layer B.Cu) (net 60))
@@
   (segment (start 37.30625 103.0375) (end 36.39375 103.95) (width 0.25) (layer F.Cu) (net 60))
   (segment (start 37.30625 93.6625) (end 37.30625 103.0375) (width 0.25) (layer F.Cu) (net 60))
+  (segment (start 188.11875 109.5375) (end 188.348501 109.767251) (width 0.25) (layer F.Cu) (net 60))
+  (segment (start 188.348501 129.151499) (end 188.348501 109.767251) (width 0.25) (layer F.Cu) (net 60))
+  (segment (start 184.94375 96.04375) (end 184.872101 96.115399) (width 0.25) (layer F.Cu) (net 60))
+  (segment (start 186.025248 109.5375) (end 188.11875 109.5375) (width 0.25) (layer F.Cu) (net 60))
+  (segment (start 184.872101 96.115399) (end 184.872101 108.384353) (width 0.25) (layer F.Cu) (net 60))
+  (segment (start 184.872101 108.384353) (end 186.025248 109.5375) (width 0.25) (layer F.Cu) (net 60))
   (segment (start 54.13375 69.69125) (end 54.13375 86.36) (width 0.25) (layer F.Cu) (net 61))
   (segment (start 54.13375 67.31) (end 54.13375 69.69125) (width 0.25) (layer F.Cu) (net 61))
@@
   (segment (start 164.30625 131.7625) (end 165.89375 133.35) (width 0.25) (layer B.Cu) (net 78))
   (segment (start 158.89375 131.525) (end 159.13125 131.7625) (width 0.25) (layer B.Cu) (net 78))
+  (zone (net 0) (net_name "") (layer B.Cu) (hatch edge 0.508)
+    (connect_pads (clearance 0.508))
+    (min_thickness 0.25)
+    (fill yes (arc_segments 32) (thermal_gap 0.508) (thermal_bridge_width 0.508))
+    (polygon
+      (pts
+        (xy 54.76875 60.325) (xy 277.01875 60.325) (xy 277.01875 137.31875) (xy 29.36875 137.31875) (xy 29.36875 60.325)
+        (xy 42.06875 60.325) (xy 42.06875 54.76875) (xy 54.76875 54.76875)
+      )
+    )
+  )
+  (zone (net 0) (net_name "") (layer F.Cu) (hatch edge 0.508)
+    (connect_pads (clearance 0.508))
+    (min_thickness 0.25)
+    (fill yes (arc_segments 32) (thermal_gap 0.508) (thermal_bridge_width 0.508))
+    (polygon
+      (pts
+        (xy 54.76875 60.325) (xy 277.01875 60.325) (xy 277.01875 137.31875) (xy 29.36875 137.31875) (xy 29.36875 60.325)
+        (xy 42.06875 60.325) (xy 42.06875 54.76875) (xy 54.76875 54.76875)
+      )
+    )
+  )
 )

Commit message: Add some cosmetic changes
Routing:
- net (no net): track 6.74 -> 285.4 mm
- net GND: track 298.7 -> 264.7 mm
- net ROW3: track 268.1 -> 264.3 mm
- net +5V: track 303.4 -> 300.4 mm
- net Net-(R3-Pad1): track 153.4 -> 150.5 mm
- net COL0: track 285.6 -> 283.2 mm
- net ROW2: track 392.9 -> 390.9 mm
- net ROW0: track 434.8 -> 432.9 mm
- net COL12: track 237.1 -> 235.2 mm
- net COL11: track 215.9 -> 214.1 mm
- net COL10: track 193.8 -> 192.0 mm
- net COL2: track 246.0 -> 244.4 mm
- net COL6: track 121.8 -> 120.7 mm
- net COL7: track 75.4 -> 74.5 mm
- removed copper zone on B.Cu, net (none)
- removed copper zone on F.Cu, net (none)

Commit message: Flip stabs
Parts:
- MX44: footprint MX_Alps_Hybrid:MX-2.75U-NoLED -> MX_Alps_Hybrid:MX-2.75U-ReversedStabilizers-NoLED
- MX46: footprint MX_Alps_Hybrid:MX-2.25U-NoLED -> MX_Alps_Hybrid:MX-2.25U-ReversedStabilizers-NoLED
Routing:
- net (no net): track 285.4 -> 359.0 mm
- net +5V: track 300.4 -> 293.4 mm
- net ROW2: track 390.9 -> 394.1 mm
- net ROW1: track 413.2 -> 415.2 mm
- net COL3: track 219.2 -> 221.2 mm
- net Net-(R1-Pad2): track 124.4 -> 126.0 mm
- net COL2: track 244.4 -> 245.6 mm
- net COL0: track 283.2 -> 282.7 mm
- added copper zone on B.Cu, net (none)
- added copper zone on F.Cu, net (none)

Commit message: Add gerber files
Parts:
- added G***: LOGO, Front_logo:shelk, F.Cu at (154.0, 99.2)
